Commit message: Finalizing Week 1 Challenge and Infrastructure for Professional Repo

File: challenges/week1/puzzlebot_sim/urdf/puzzlebot.urdf (robot description, URDF)
Before this commit: robot Puzzlebot_Jetson_Lidar_Ed., 0 links, 0 joints
Links:
- added link base_footprint
- added link base_link; visual mesh filename=package://puzzlebot_sim/meshes/Puzzlebot_Jetson_Lidar_Editi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
- added link caster_link; visual mesh filename=package://puzzlebot_sim/meshes/Puzzlebot_Caster_Wheel.stl
- added link wheel_l_link; visual mesh filename=package://puzzlebot_sim/meshes/Puzzlebot_Wheel.stl
- added link wheel_r_link; visual mesh filename=package://puzzlebot_sim/meshes/Puzzlebot_Wheel.stl
Joints:
- added joint base_link_joint: type fixed, parent base_footprint, child base_link, origin xyz=0 0 0.05 rpy=0 0 0
- added joint caster_joint: type fixed, parent base_link, child caster_link, origin xyz=-0.095 0 -0.03 rpy=0 0 0
- added joint wheel_l_joint: type continuous, parent base_link, child wheel_l_link, origin xyz=0.052 0.095 -0.0025 rpy=0 0 0, axis 0 1 0
- added joint wheel_r_joint: type continuous, parent base_link, child wheel_r_link, origin xyz=0.052 -0.095 -0.0025 rpy=0 0 0, axis 0 1 0

Commit message: feat: Week 1 Challenge - Kinematic simulation with TF and terminal logging

File: challenges/week1/puzzlebot_sim/urdf/puzzlebot.urdf (robot description, URDF)
Before this commit: robot Puzzlebot_Jetson_Lidar_Ed., 5 links, 4 joints
Joints:
- joint base_link_joint: origin xyz=0 0 0.05 rpy=0 0 0 -> xyz=0.0 0.0 0.05 rpy=0 0 0
- joint caster_joint: origin xyz=-0.095 0 -0.03 rpy=0 0 0 -> xyz=-0.095 0.0 -0.03 rpy=0 0 0

Commit message: feat: finalize puzzlebot simulation setup, rviz config, and tf report generation

File: challenges/week1/puzzlebot_sim/urdf/puzzlebot.urdf (robot description, URDF)
Before this commit: robot Puzzlebot_Jetson_Lidar_Ed., 5 links, 4 joints
Links:
- removed link caster_link
- removed link wheel_l_link
- removed link wheel_r_link
- added link caster; visual mesh filename=package://puzzlebot_sim/meshes/Puzzlebot_Caster_Wheel.stl
- added link wheel_l; visual mesh filename=package://puzzlebot_sim/meshes/Puzzlebot_Wheel.stl
- added link wheel_r; visual mesh filename=package://puzzlebot_sim/meshes/Puzzlebot_Wheel.stl
Joints:
- joint caster_joint: child caster_link -> caster
- joint wheel_l_joint: child wheel_l_link -> wheel_l; origin xyz=0.052 0.095 -0.0025 rpy=0 0 0 -> xyz=0.0 0.09 0.0 rpy=0 0 0
- joint wheel_r_joint: axis 0 1 0 -> 0 -1 0; child wheel_r_link -> wheel_r; origin xyz=0.052 -0.095 -0.0025 rpy=0 0 0 -> xyz=0.0 -0.09 0.0 rpy=0 0 3.14159
